File: Leiterplatte/mini-sps-leiterplatte-kicad/mini-sps-leiterplatte-kicad.kicad_sch (KiCad schematic)
At the start: 17 parts, among them J1 Conn_01x03_Socket, J2 Conn_01x03_Socket, J3 Conn_01x03_Socket, K1 SRD-05VDC-SL-C, K2 SRD-05VDC-SL-C, K3 SRD-05VDC-SL-C

Commit message: v.2 schreubdinger
Parts:
- added J4: Conn_01x03_Socket, TerminalBlock:TerminalBlock_Altech_AK300-3_P5.00mm, symbol Connector:Conn_01x03_Socket
- added J6, J7: Conn_01x02_Socket, TerminalBlock:TerminalBlock_Altech_AK300-2_P5.00mm, symbol Connector:Conn_01x02_Socket
- D1, D2, D3: footprint (none) -> LED_THT:LED_D5.0mm
- D4: footprint (none) -> LED_THT:LED_D5.0mm-4_RGB_Wide_Pins
- J1, J2, J3: footprint (none) -> TerminalBlock:TerminalBlock_Altech_AK300-3_P5.00mm
- K1, K2, K3: footprint SRD-05VDC-SL-C:RELAY_SRD-05VDC-SL-C -> custom:RELAY_SRD-05VDC-SL-C
- R1, R2, R3, R4, R5, R6: footprint (none) -> Resistor_THT:R_Axial_DIN0207_L6.3mm_D2.5mm_P10.16mm_Horizontal
Connections:
- net GND: now also A1.29 (GND), A1.4 (GND), J6.2 (Pin_2)
- net D8: now reaches A1.11 (D8)
- net D8: now also J4.1 (Pin_1)
- net D9: now reaches A1.12 (D9)
- net D9: now also J4.2 (Pin_2)
- net D10: now reaches A1.13 (D10)
- net D10: now also J4.3 (Pin_3)
- net A0: now reaches A1.19 (A0)
- net A0: now also J7.1 (Pin_1)
- net A1: now reaches A1.20 (A1)
- net A1: now also J7.2 (Pin_2)
- net at A1.30 (VIN): now also J6.1 (Pin_1)
Other:
- note added: "Arduino Nano+Spannungsversorgung"
- note added: "DIO-Schutzschaltung"
- note added: "Schutzschaltung AI"

Commit message: v.3 Spannungsversorgung etc
Parts:
- removed A1: Arduino_Nano_Every, Module:Arduino_Nano, symbol MCU_Module:Arduino_Nano_Every
- removed J6: Conn_01x02_Socket, TerminalBlock:TerminalBlock_Altech_AK300-2_P5.00mm, symbol Connector:Conn_01x02_Socket
- added A1: Arduino_Nano_v3.x, Module:Arduino_Nano, symbol MCU_Module:Arduino_Nano_v3.x
- added C1, C2: C, symbol Device:C
- added C3: C_Polarized, symbol Device:C_Polarized
- added D10, D13, D7: LED, symbol Device:LED
- added D11, D12, D5, D6, D8, D9: D_Zener, symbol Device:D_Zener
- added D14: 1N4007, symbol Device:D
- added J5: Conn_01x03_Socket, TerminalBlock:TerminalBlock_Altech_AK300-3_P5.00mm, symbol Connector:Conn_01x03_Socket
- added R10, R12: 39k, symbol Device:R
- added R11, R13: 10k, symbol Device:R
- added R7, R8, R9: R, symbol Device:R
- added U1: L7805, symbol Regulator_Linear:L7805
Connections:
- net D4 is gone; now on net D3: K3.A2, R3.2
- net A0: now also A1.19 (A0), R10.1; no longer J7.1 (Pin_1)
- net A1: now also A1.20 (A1), R12.1; no longer J7.2 (Pin_2)
- net D10: now also A1.13 (D10), J5.1 (Pin_1); no longer J4.3 (Pin_3)
- net D2: now also K2.A2, R2.2, A1.5 (D2); no longer K1.A2, R1.2
- net D3: now also A1.6 (D3); no longer K2.A2, R2.2
- net D8: now also A1.11 (D8), D8.2 (A), D9.1 (K), R8.1; no longer J4.1 (Pin_1)
- net D9: now also A1.12 (D9), D11.2 (A), D12.1 (K), R9.1; no longer J4.2 (Pin_2)
- net GND: now also A1.4 (GND), C1.2, C2.2, C3.2, D10.1 (K), D12.2 (A), D13.1 (K), D5.2 (A), D7.1 (K), D9.2 (A), R11.2, R13.2, U1.2 (GND)
- net D5(R) renamed D4(R)
- net D4(R): now also A1.7 (D4)
- net D6(G) renamed D5(G)
- net D5(G): now also A1.8 (D5)
- net D7(B) renamed D6(B)
- net D6(B): now also A1.9 (D6)
- new net: J7.1 (Pin_1), R10.2, R11.1
- new net: C2.1, C3.1, D14.1 (K), U1.1 (IN)
- new net: D11.1 (K), J4.1 (Pin_1)
- new net: D10.2 (A), R8.2
- new net: D7.2 (A), R7.2
- new net: D6.1 (K), J4.3 (Pin_3)
- new net: D8.1 (K), J4.2 (Pin_2)
- new net: J7.2 (Pin_2), R12.2, R13.1
- new net: D13.2 (A), R9.2
- new net 5V: A1.30 (VIN), C1.1, D14.2 (A), U1.3 (OUT)
- new net D1: A1.1 (D1/TX), K1.A2, R1.2
- new net D11: A1.14 (D11), J5.2 (Pin_2)
- new net D12: A1.15 (D12), J5.3 (Pin_3)
- new net D7: A1.10 (D7), D5.1 (K), D6.2 (A), R7.1
Other:
- note added: "Arduino Nano"
- note added: "DI-Schutzschaltung"
- note added: "DO-Schutzschaltung //to do"
- note removed: "Arduino Nano+Spannungsversorgung"
- note removed: "DIO-Schutzschaltung"
- moved on the sheet: D1, D2, D3, D4, J1, J2, J3, J4, J7, K1, K2, K3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

Commit message: v.4 footprints):
Parts:
- removed J1, J2, J3, J4, J5: Conn_01x03_Socket, TerminalBlock:TerminalBlock_Altech_AK300-3_P5.00mm, symbol Connector:Conn_01x03_Socket
- removed J7: Conn_01x02_Socket, TerminalBlock:TerminalBlock_Altech_AK300-2_P5.00mm, symbol Connector:Conn_01x02_Socket
- added J1, J2, J3, J4, J6: Screw_Terminal_01x03, TerminalBlock:TerminalBlock_bornier-3_P5.08mm, symbol Connector:Screw_Terminal_01x03
- added J5, J7: Screw_Terminal_01x02, TerminalBlock:TerminalBlock_bornier-2_P5.08mm, symbol Connector:Screw_Terminal_01x02
- C1: value C -> 100nF; footprint (none) -> Capacitor_THT:C_Disc_D7.0mm_W2.5mm_P5.00mm
- C2: value C -> 330 nF; footprint (none) -> Capacitor_THT:C_Disc_D7.0mm_W2.5mm_P5.00mm
- C3: value C_Polarized -> 10uF; footprint (none) -> Capacitor_THT:CP_Radial_D13.0mm_P5.00mm
- D10, D13, D7: footprint (none) -> LED_THT:LED_D5.0mm
- D11, D12, D14, D5, D6, D8, D9: footprint (none) -> Diode_THT:D_DO-15_P15.24mm_Horizontal
- R10, R11, R12, R13, R7, R8, R9: footprint (none) -> Resistor_THT:R_Axial_DIN0207_L6.3mm_D2.5mm_P10.16mm_Horizontal
- U1: footprint (none) -> Package_TO_SOT_THT:TO-220-3_Vertical
Connections:
- net D10: now also J4.1 (Pin_1)
- net D11: now also J4.2 (Pin_2)
- net D12: now also J4.3 (Pin_3)
- net GND: now also J7.1 (Pin_1)
- net at R10.2, R11.1: now also J5.1 (Pin_1)
- net at K3.NO: now also J6.1 (Pin_1)
- net at K3.COM: now also J6.2 (Pin_2)
- net at K3.NC: now also J6.3 (Pin_3)
- net at C2.1, C3.1, D14.1 (K)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: now also J7.2 (Pin_2)
- net at K2.NO: now also J2.1 (Pin_1)
- net at K2.COM: now also J2.2 (Pin_2)
- net at K2.NC: now also J2.3 (Pin_3)
- net at D11.1 (K): now also J3.1 (Pin_1)
- net at D6.1 (K): now also J3.3 (Pin_3)
- net at D8.1 (K): now also J3.2 (Pin_2)
- net at R12.2, R13.1: now also J5.2 (Pin_2)
- net at K1.NO: now also J1.1 (Pin_1)
- net at K1.COM: now also J1.2 (Pin_2)
- net at K1.NC: now also J1.3 (Pin_3)
Other:
- note added: "Spannungswandler"
- moved on the sheet: D7, R8

Commit message: alles auf den neusten fucking stand
Parts:
- removed D1, D10, D13, D2, D7: LED, LED_THT:LED_D5.0mm, symbol Device:LED
- removed D4: LED_RGB, LED_THT:LED_D5.0mm-4_RGB_Wide_Pins, symbol Device:LED_RGB
- removed J1, J2, J3, J4, J6: Screw_Terminal_01x03, TerminalBlock:TerminalBlock_bornier-3_P5.08mm, symbol Connector:Screw_Terminal_01x03
- removed J5, J7: Screw_Terminal_01x02, TerminalBlock:TerminalBlock_bornier-2_P5.08mm, symbol Connector:Screw_Terminal_01x02
- removed K3: SRD-05VDC-SL-C, custom:RELAY_SRD-05VDC-SL-C, symbol custom:SRD-05VDC-SL-C
- added D1, D2: 1N4007, Diode_THT:D_DO-15_P15.24mm_Horizontal, symbol Device:D
- added D4, D5: LED, LED_THT:LED_D5.0mm, symbol Device:LED
- added J1: Screw_Terminal_01x16, TerminalBlock_CUI:TerminalBlock_CUI_TB007-508-16_1x16_P5.08mm_Horizontal, symbol Connector:Screw_Terminal_01x16
- added Q1, Q2: BC547, Package_TO_SOT_THT:TO-92L_Inline_Wide, symbol Transistor_BJT:BC547
- added R0: 0, Resistor_THT:R_Axial_DIN0207_L6.3mm_D2.5mm_P10.16mm_Horizontal, symbol Device:R
- R1, R2: value 330 -> 1k
- R3: value 330 -> 0
- R7, R8, R9: value R -> 0
- renumbered D5 to D7
Connections:
- net 5V: now also K1.A2, K2.A2, D1.2 (A), D2.2 (A), J1.15 (Pin_15), J1.16 (Pin_16), R0.1, R0.2
- net D1: no longer K1.A2
- net D2: no longer K2.A2
- net D3: no longer R3.2
- net D7: no longer R7.1
- net D8: no longer R8.1
- net D9: no longer R9.1
- net GND: now also A1.29 (GND), R3.1, R3.2, R7.1, R7.2, R8.1, R8.2, R9.1, R9.2, D4.1 (K), D5.1 (K), J1.10 (Pin_10), J1.8 (Pin_8), Q1.3 (E), Q2.3 (E); no longer K1.A1, K2.A1
- net at R6.2: now also D5.2 (A)
- net at R5.2: now also D4.2 (A)
- net at R4.2: now also D3.2 (A)
- net AIN 1: now reaches R10.2, R11.1
- net AIN 1: now also J1.7 (Pin_7)
- net Vin: now reaches C2.1, C3.1, D14.1 (K), U1.1 (IN)
- net Vin: now also J1.11 (Pin_11)
- net AIN 2: now reaches R12.2, R13.1
- net AIN 2: now also J1.9 (Pin_9)
- net DI3: now reaches D11.1 (K)
- net DI3: now also J1.14 (Pin_14)
- net DI1: now reaches D6.1 (K)
- net DI1: now also J1.12 (Pin_12)
- net NO 1: now reaches K1.NO
- net NO 1: now also J1.3 (Pin_3)
- net COM1: now reaches K1.COM
- net COM1: now also J1.2 (Pin_2)
- net NC 1: now reaches K1.NC
- net NC 1: now also J1.1 (Pin_1)
- net DI2: now reaches D8.1 (K)
- net DI2: now also J1.13 (Pin_13)
- net at R1.1: now also Q1.2 (B)
- net at R2.1: now also Q2.2 (B)
- net COM2: now reaches K2.COM
- net COM2: now also J1.5 (Pin_5)
- net NC 2: now reaches K2.NC
- net NC 2: now also J1.4 (Pin_4)
- net NO 2: now reaches K2.NO
- net NO 2: now also J1.6 (Pin_6)
- new net: D2.1 (K), K2.A1, Q2.1 (C)
- new net: D1.1 (K), K1.A1, Q1.1 (C)
Other:
- note added: "Brücken"
- note added: "Screwterminal"
- note removed: "DO-Schutzschaltung //to do"
- moved on the sheet: A1, C1, C2, C3, D14, K1, R10, R11, R12, R13, R4, R5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

Commit message: fertig lk
Connections:
- net 5V: no longer A1.30 (VIN), C1.1, D1.2 (A), D14.2 (A), D2.2 (A), K1.A2, K2.A2, R0.1, R0.2, U1.3 (OUT)
- net D10: no longer names the net of A1.13 (D10)
- net D11: no longer names the net of A1.14 (D11)
- net D12: no longer names the net of A1.15 (D12)
- net D3: no longer names the net of A1.6 (D3)
- new net +5V: A1.30 (VIN), C1.1, D1.2 (A), D14.2 (A), D2.2 (A), K1.A2, K2.A2, R0.1, R0.2, U1.3 (OUT)
- no-connect marks 0 -> 17
Other:
- moved on the sheet: D3, D4, D5, R4, R5, R6, R8, R9
