File: Leiterplatte/mini-sps-leiterplatte-kicad/mini-sps-leiterplatte-kicad.kicad_pcb (KiCad board)
At the start: 2 copper layers, 20 parts, among them J1 Conn_01x03_Socket, J2 Conn_01x03_Socket, J3 Conn_01x03_Socket, J4 Conn_01x03_Socket, J6 Conn_01x02_Socket, J7 Conn_01x02_Socket, K1 SRD-05VDC-SL-C, K2 SRD-05VDC-SL-C, K3 SRD-05VDC-SL-C

Commit message: v.4 footprints):
Parts:
- added C1: 100nF, Capacitor_THT:C_Disc_D7.0mm_W2.5mm_P5.00mm, F.Cu at (174.0, 73.7)
- added C2: 330 nF, Capacitor_THT:C_Disc_D7.0mm_W2.5mm_P5.00mm, F.Cu at (191.8, 73.7)
- added C3: 10uF, Capacitor_THT:CP_Radial_D13.0mm_P5.00mm, F.Cu at (182.9, 83.7)
- added D10: LED, LED_THT:LED_D5.0mm, F.Cu at (79.0, 165.1)
- added D11: D_Zener, Diode_THT:D_DO-15_P15.24mm_Horizontal, F.Cu at (-48.4, 94.0)
- added D12: D_Zener, Diode_THT:D_DO-15_P15.24mm_Horizontal, F.Cu at (-43.2, 94.0)
- added D13: LED, LED_THT:LED_D5.0mm, F.Cu at (79.0, 172.6)
- added D14: 1N4007, Diode_THT:D_DO-15_P15.24mm_Horizontal, F.Cu at (-38.1, 94.0)
- added D5: D_Zener, Diode_THT:D_DO-15_P15.24mm_Horizontal, F.Cu at (175.3, 91.4)
- added D6: D_Zener, Diode_THT:D_DO-15_P15.24mm_Horizontal, F.Cu at (-63.9, 94.0)
- added D7: LED, LED_THT:LED_D5.0mm, F.Cu at (79.0, 157.7)
- added D8: D_Zener, Diode_THT:D_DO-15_P15.24mm_Horizontal, F.Cu at (-58.7, 94.0)
- added D9: D_Zener, Diode_THT:D_DO-15_P15.24mm_Horizontal, F.Cu at (-53.5, 94.0)
- added J5: Screw_Terminal_01x02, TerminalBlock:TerminalBlock_bornier-2_P5.08mm, F.Cu at (125.7, 165.1)
- added R10: 39k, Resistor_THT:R_Axial_DIN0207_L6.3mm_D2.5mm_P10.16mm_Horizontal, F.Cu at (64.8, 168.1)
- added R11: 10k, Resistor_THT:R_Axial_DIN0207_L6.3mm_D2.5mm_P10.16mm_Horizontal, F.Cu at (64.8, 172.2)
- added R12: 39k, Resistor_THT:R_Axial_DIN0207_L6.3mm_D2.5mm_P10.16mm_Horizontal, F.Cu at (64.8, 176.2)
- added R13: 10k, Resistor_THT:R_Axial_DIN0207_L6.3mm_D2.5mm_P10.16mm_Horizontal, F.Cu at (64.8, 180.2)
- added R7: R, Resistor_THT:R_Axial_DIN0207_L6.3mm_D2.5mm_P10.16mm_Horizontal, F.Cu at (64.8, 155.9)
- added R8: R, Resistor_THT:R_Axial_DIN0207_L6.3mm_D2.5mm_P10.16mm_Horizontal, F.Cu at (64.8, 160.0)
- added R9: R, Resistor_THT:R_Axial_DIN0207_L6.3mm_D2.5mm_P10.16mm_Horizontal, F.Cu at (64.8, 164.1)
- added U1: L7805, Package_TO_SOT_THT:TO-220-3_Vertical, F.Cu at (186.7, 69.8)
- A1: value Arduino_Nano_Every -> Arduino_Nano_v3.x
- J1, J2, J3, J4: value Conn_01x03_Socket -> Screw_Terminal_01x03; footprint TerminalBlock:TerminalBlock_Altech_AK300-3_P5.00mm -> TerminalBlock:TerminalBlock_bornier-3_P5.08mm
- J6: value Conn_01x02_Socket -> Screw_Terminal_01x03; footprint TerminalBlock:TerminalBlock_Altech_AK300-2_P5.00mm -> TerminalBlock:TerminalBlock_bornier-3_P5.08mm
- J7: value Conn_01x02_Socket -> Screw_Terminal_01x02; footprint TerminalBlock:TerminalBlock_Altech_AK300-2_P5.00mm -> TerminalBlock:TerminalBlock_bornier-2_P5.08mm
- moved D4 210.8 mm to (16.1, 181.6), turned to 0 degrees
- moved J6 186.8 mm to (42.9, 173.1), turned to 0 degrees
- moved R5 185.1 mm to (16.1, 149.3), turned to 0 degrees
- moved R6 178.1 mm to (16.1, 153.4), turned to 0 degrees
- moved R4 174.8 mm to (16.1, 145.3), turned to 0 degrees
- moved J4 168.7 mm to (42.9, 164.1), turned to 0 degrees
- moved J7 151.2 mm to (59.6, 145.9), turned to 0 degrees
- moved D1 145.6 mm to (17.0, 159.2), turned to 0 degrees
- moved D2 139.5 mm to (17.0, 166.6), turned to 0 degrees
- moved R1 137.3 mm to (16.1, 133.1), turned to 0 degrees
- moved D3 133.9 mm to (17.0, 174.1), turned to 0 degrees
- moved R2 131.6 mm to (16.1, 137.2), turned to 0 degrees
- moved R3 127.5 mm to (16.1, 141.2), turned to 0 degrees
- moved J1 94.8 mm to (42.9, 136.9), turned to 0 degrees
- moved J2 90.1 mm to (42.9, 145.9), turned to 0 degrees
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Connections:
- A1 pad 1: unconnected-(A1-TX1-Pad1) -> D1
- A1 pad 10: D7(B) -> D7
- A1 pad 14: unconnected-(A1-MOSI-Pad14) -> D11
- A1 pad 15: unconnected-(A1-MISO-Pad15) -> D12
- A1 pad 29: GND -> unconnected-(A1-GND-Pad29)
- A1 pad 30: Net-(A1-VIN) -> 5V
- A1 pad 7: D4 -> D4(R)
- A1 pad 8: D5(R) -> D5(G)
- A1 pad 9: D6(G) -> D6(B)
- J3 pad 1: Net-(J3-Pin_1) -> Net-(D11-K)
- J3 pad 2: Net-(J3-Pin_2) -> Net-(D8-K)
- J3 pad 3: Net-(J3-Pin_3) -> Net-(D6-K)
- J4 pad 1: D8 -> D10
- J4 pad 2: D9 -> D11
- J4 pad 3: D10 -> D12
- J6 pad 1: Net-(A1-VIN) -> Net-(J6-Pin_1)
- J6 pad 2: GND -> Net-(J6-Pin_2)
- J7 pad 1: A0 -> GND
- J7 pad 2: A1 -> Net-(D14-K)
- K1 pad A2: D2 -> D1
- K2 pad A2: D3 -> D2
- K3 pad A2: D4 -> D3
- K3 pad COM: Net-(J3-Pin_2) -> Net-(J6-Pin_2)
- K3 pad NC: Net-(J3-Pin_3) -> Net-(J6-Pin_3)
- K3 pad NO: Net-(J3-Pin_1) -> Net-(J6-Pin_1)
- R1 pad 2: D2 -> D1
- R2 pad 2: D3 -> D2
- R3 pad 2: D4 -> D3
- R4 pad 1: D5(R) -> D4(R)
- R5 pad 1: D6(G) -> D5(G)
- R6 pad 1: D7(B) -> D6(B)
Other:
- board outline added: 150.5 x 85.5 mm

Commit message: alles auf den neusten fucking stand
Parts:
- removed D13: LED, LED_THT:LED_D5.0mm
- removed D14: 1N4007, Diode_THT:D_DO-15_P15.24mm_Horizontal
- removed J2, J3, J4, J6: Screw_Terminal_01x03, TerminalBlock:TerminalBlock_bornier-3_P5.08mm
- removed J5, J7: Screw_Terminal_01x02, TerminalBlock:TerminalBlock_bornier-2_P5.08mm
- removed K3: SRD-05VDC-SL-C, custom:RELAY_SRD-05VDC-SL-C
- added Q1: BC547, Package_TO_SOT_THT:TO-92L_Inline_Wide, F.Cu at (142.8, 113.0)
- added Q2: BC547, Package_TO_SOT_THT:TO-92L_Inline_Wide, F.Cu at (150.4, 112.8)
- added R14: 0, Resistor_THT:R_Axial_DIN0207_L6.3mm_D2.5mm_P10.16mm_Horizontal, F.Cu at (130.0, 122.9)
- D1, D10: value LED -> D_Zener; footprint LED_THT:LED_D5.0mm -> Diode_THT:D_DO-15_P15.24mm_Horizontal
- D2, D7: value LED -> 1N4007; footprint LED_THT:LED_D5.0mm -> Diode_THT:D_DO-15_P15.24mm_Horizontal
- D4: value LED_RGB -> LED; footprint LED_THT:LED_D5.0mm-4_RGB_Wide_Pins -> LED_THT:LED_D5.0mm
- D5: value D_Zener -> LED; footprint Diode_THT:D_DO-15_P15.24mm_Horizontal -> LED_THT:LED_D5.0mm
- D8: value D_Zener -> 1N4007
- J1: value Screw_Terminal_01x03 -> Screw_Terminal_01x16; footprint TerminalBlock:TerminalBlock_bornier-3_P5.08mm -> TerminalBlock_CUI:TerminalBlock_CUI_TB007-508-16_1x16_P5.08mm_Horizontal
- R1, R3: value 330 -> 0
- R10: value 39k -> 1k
- R11: value 10k -> 0
- R2: value 330 -> 39k
- R5: value 330 -> 10k
- R7: value R -> 330
- R8: value R -> 0
- R9: value R -> 1k
- moved D8 245.1 mm to (186.0, 108.0), turned to 180 degrees
- moved D6 190.9 mm to (126.3, 110.5)
- moved D12 178.6 mm to (134.1, 115.3), turned to -90 degrees
- moved D11 177.0 mm to (125.0, 129.5)
- moved D9 172.1 mm to (114.9, 129.5)
- moved D2 171.4 mm to (160.0, 72.1), turned to 180 degrees
- moved R13 146.4 mm to (185.4, 97.2), turned to 180 degrees
- moved J1 138.0 mm to (180.9, 138.4), turned to 180 degrees
- moved R12 133.6 mm to (175.3, 101.0)
- moved R2 126.7 mm to (132.7, 87.6), turned to -90 degrees
- moved R5 126.5 mm to (132.7, 100.3), turned to -90 degrees
- moved R6 123.0 mm to (122.5, 91.7), turned to 180 degrees
- moved R11 122.5 mm to (162.1, 97.5)
- moved D4 121.9 mm to (106.0, 99.2)
- moved D3 121.3 mm to (106.0, 91.7)
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Connections:
- A1 pad 29: unconnected-(A1-GND-Pad29) -> GND
- C2 pad 1: Net-(D14-K) -> Vin
- C3 pad 1: Net-(D14-K) -> Vin
- D1 pad 1: GND -> D8
- D1 pad 2: Net-(D1-A) -> GND
- D10 pad 1: GND -> DI2
- D10 pad 2: Net-(D10-A) -> D8
- D11 pad 1: Net-(D11-K) -> DI1
- D11 pad 2: D9 -> D7
- D2 pad 1: GND -> Vin
- D2 pad 2: Net-(D2-A) -> 5V
- D4 pad 2: GND -> Net-(D4-A)
- D5 pad 1: D7 -> GND
- D5 pad 2: GND -> Net-(D5-A)
- D6 pad 1: Net-(D6-K) -> D7
- D6 pad 2: D7 -> GND
- D7 pad 1: GND -> Net-(D2-K)
- D7 pad 2: Net-(D7-A) -> 5V
- D8 pad 1: Net-(D8-K) -> Net-(D1-K)
- D8 pad 2: D8 -> 5V
- D9 pad 1: D8 -> DI3
- D9 pad 2: GND -> D9
- J1 pad 1: Net-(J1-Pin_1) -> NC 1
- J1 pad 2: Net-(J1-Pin_2) -> COM1
- J1 pad 3: Net-(J1-Pin_3) -> NO 1
- K1 pad A1: GND -> Net-(D2-K)
- K1 pad A2: D1 -> 5V
- K1 pad COM: Net-(J1-Pin_2) -> COM2
- K1 pad NC: Net-(J1-Pin_3) -> NC 2
- K1 pad NO: Net-(J1-Pin_1) -> NO 2
- K2 pad A1: GND -> Net-(D1-K)
- K2 pad A2: D2 -> 5V
- K2 pad COM: Net-(J2-Pin_2) -> COM1
- K2 pad NC: Net-(J2-Pin_3) -> NC 1
- K2 pad NO: Net-(J2-Pin_1) -> NO 1
- R1 pad 1: Net-(D1-A) -> GND
- R1 pad 2: D1 -> GND
- R10 pad 1: A0 -> Net-(Q2-B)
- R10 pad 2: Net-(J5-Pin_1) -> D2
- R11 pad 1: Net-(J5-Pin_1) -> GND
- R12 pad 1: A1 -> A0
- R12 pad 2: Net-(J5-Pin_2) -> AIN 1
- R13 pad 1: Net-(J5-Pin_2) -> AIN 1
- R2 pad 1: Net-(D2-A) -> A1
- R2 pad 2: D2 -> AIN 2
- R3 pad 1: Net-(D3-A) -> GND
- R3 pad 2: D3 -> GND
- R4 pad 1: D4(R) -> D6(B)
- R4 pad 2: Net-(D4-RA) -> Net-(D5-A)
- R5 pad 1: D5(G) -> AIN 2
- R5 pad 2: Net-(D4-GA) -> GND
- R6 pad 1: D6(B) -> D4(R)
- R6 pad 2: Net-(D4-BA) -> Net-(D3-A)
- R7 pad 1: D7 -> D5(G)
- R7 pad 2: Net-(D7-A) -> Net-(D4-A)
- R8 pad 1: D8 -> 5V
- R8 pad 2: Net-(D10-A) -> 5V
- R9 pad 1: D9 -> Net-(Q1-B)
- R9 pad 2: Net-(D13-A) -> D1
- U1 pad 1: Net-(D14-K) -> Vin
Routing:
- net GND: track 0.00 -> 393.9 mm, vias 0 -> 12
- net 5V: track 0.00 -> 289.4 mm
- net D9: track 0.00 -> 217.0 mm
- net Vin: track 0.00 -> 192.4 mm
- net AIN 2: track 0.00 -> 111.2 mm
- net AIN 1: track 0.00 -> 85.5 mm
- net D8: track 0.00 -> 84.2 mm
- net Net-(D1-K): track 0.00 -> 75.0 mm
- net D5(G): track 0.00 -> 53.9 mm
- net D6(B): track 0.00 -> 53.7 mm
- net D7: track 0.00 -> 49.3 mm
- net A1: track 0.00 -> 38.7 mm
- net D4(R): track 0.00 -> 38.0 mm
- net A0: track 0.00 -> 35.7 mm
- net Net-(D2-K): track 0.00 -> 34.5 mm
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- added copper zone on B.Cu, net GND
Other:
- board size 150.5 x 85.5 mm -> 100 x 100 mm
- board text added: "Katrin F. Cedric S. Linda S."
- board text added: "Riesen SPS"

Commit message: fertig lk
Parts:
- renumbered D8 to D1, D9 to D11, D2 to D14, D7 to D2, D11 to D6, D6 to D7, D10 to D8, D1 to D9, K2 to K1, K1 to K2, R8 to R0, R9 to R1, R12 to R10, R13 to R11, R2 to R12, R5 to R13, R10 to R2, R6 to R4, R7 to R5, R4 to R6, R14 to R7, R11 to R8, R1 to R9
Connections:
- net 5V renamed +5V
- A1 pad 13: D10 -> unconnected-(A1-D10-Pad13)
- A1 pad 14: D11 -> unconnected-(A1-D11-Pad14)
- A1 pad 15: D12 -> unconnected-(A1-D12-Pad15)
- A1 pad 6: D3 -> unconnected-(A1-D3-Pad6)
Routing:
- net Vin: track 192.4 -> 190.4 mm
- net GND: vias 12 -> 0
- net (no net): vias 1 -> 4

Commit message: version 2
Parts:
- removed R0, R9: 0, Resistor_THT:R_Axial_DIN0207_L6.3mm_D2.5mm_P10.16mm_Horizontal
- removed R12: 39k, Resistor_THT:R_Axial_DIN0207_L6.3mm_D2.5mm_P10.16mm_Horizontal
- removed R13: 10k, Resistor_THT:R_Axial_DIN0207_L6.3mm_D2.5mm_P10.16mm_Horizontal
- added D10: LED, LED_THT:LED_D5.0mm, F.Cu at (109.5, 111.6)
- added D13: LED, LED_THT:LED_D5.0mm, F.Cu at (125.5, 111.6)
- added D15: BZV55B5V1, Diode_THT:D_DO-35_SOD27_P10.16mm_Horizontal, F.Cu at (141.4, 101.1)
- added R14: 1500, Resistor_THT:R_Axial_DIN0207_L6.3mm_D2.5mm_P10.16mm_Horizontal, F.Cu at (127.4, 93.1)
- added R15: 10k, Resistor_THT:R_Axial_DIN0207_L6.3mm_D2.5mm_P10.16mm_Horizontal, F.Cu at (171.6, 55.1)
- added R16: 1500, Resistor_THT:R_Axial_DIN0207_L6.3mm_D2.5mm_P10.16mm_Horizontal, F.Cu at (127.4, 97.1)
- added R17: 10k, Resistor_THT:R_Axial_DIN0207_L6.3mm_D2.5mm_P10.16mm_Horizontal, F.Cu at (171.6, 61.1)
- added R19: 1500, Resistor_THT:R_Axial_DIN0207_L6.3mm_D2.5mm_P10.16mm_Horizontal, F.Cu at (127.5, 101.1)
- added R21: 10k, Resistor_THT:R_Axial_DIN0207_L6.3mm_D2.5mm_P10.16mm_Horizontal, F.Cu at (171.6, 67.1)
- added U2: PC817, Package_DIP:DIP-4_W7.62mm, F.Cu at (171.2, 95.9)
- added U3: PC817, Package_DIP:DIP-4_W7.62mm, F.Cu at (164.5, 96.1)
- added U4: PC817, Package_DIP:DIP-4_W7.62mm, F.Cu at (157.2, 95.9)
- D11, D9: value D_Zener -> BZV55B5V1; footprint Diode_THT:D_DO-15_P15.24mm_Horizontal -> Diode_THT:D_DO-35_SOD27_P10.16mm_Horizontal
- D12, D6, D8: value D_Zener -> 1N4148WT; footprint Diode_THT:D_DO-15_P15.24mm_Horizontal -> Diode_THT:D_DO-35_SOD27_P10.16mm_Horizontal
- D7: value D_Zener -> LED; footprint Diode_THT:D_DO-15_P15.24mm_Horizontal -> LED_THT:LED_D5.0mm
- K1, K2: footprint custom:RELAY_SRD-05VDC-SL-C -> relay:RELAY_SRD-05VDC-SL-C
- moved R3 77.9 mm to (190.1, 86.6), turned to 180 degrees
- moved R7 70.9 mm to (150.5, 55.0), turned to -90 degrees
- moved D5 57.7 mm to (143.5, 63.1), turned to 180 degrees
- moved U1 55.6 mm to (144.4, 112.6), turned to 0 degrees
- moved R11 51.8 mm to (145.5, 130.2), turned to 90 degrees
- moved C1 51.5 mm to (162.0, 103.1)
- moved C2 49.7 mm to (142.5, 116.1)
- moved D4 46.3 mm to (143.5, 72.1), turned to 180 degrees
- moved Q1 46.2 mm to (187.5, 101.1)
- moved D11 45.1 mm to (141.4, 93.1), turned to 0 degrees
- moved C3 43.0 mm to (133.5, 124.1)
- moved R2 40.5 mm to (171.6, 77.1), turned to 180 degrees
- moved R1 40.3 mm to (171.6, 81.1), turned to 180 degrees
- moved D3 39.0 mm to (143.5, 81.1), turned to 180 degrees
- moved D14 35.7 mm to (147.6, 105.6)
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Connections:
- D1 pad 1: Net-(D1-K) -> +5V
- D1 pad 2: +5V -> Net-(D1-A)
- D11 pad 1: DI3 -> Net-(D11-K)
- D11 pad 2: D9 -> Net-(D11-A)
- D12 pad 1: D9 -> Net-(D12-K)
- D12 pad 2: GND -> DI1
- D2 pad 1: Net-(D2-K) -> +5V
- D2 pad 2: +5V -> Net-(D2-A)
- D6 pad 1: DI1 -> Net-(D6-K)
- D6 pad 2: D7 -> DI2
- D7 pad 1: D7 -> Net-(D7-K)
- D7 pad 2: GND -> Net-(D6-K)
- D8 pad 1: DI2 -> Net-(D10-A)
- D8 pad 2: D8 -> DI3
- D9 pad 1: D8 -> Net-(D9-K)
- D9 pad 2: GND -> Net-(D9-A)
- J1 pad 7: AIN 1 -> GND1
- J1 pad 8: GND -> AIN 1
- J1 pad 9: AIN 2 -> GND
- K1 pad A1: Net-(D1-K) -> Net-(D1-A)
- K2 pad A1: Net-(D2-K) -> Net-(D2-A)
- Q1 pad 1: Net-(D1-K) -> Net-(D1-A)
- Q2 pad 1: Net-(D2-K) -> Net-(D2-A)
- R8 pad 1: GND -> GND1
- R8 pad 2: GND -> GND1
Routing:
- net GND: track 393.9 -> 192.8 mm
- net Vin: track 190.4 -> 41.4 mm
- net D9: track 217.0 -> 85.8 mm
- net GND1: track 0.00 -> 118.1 mm
- net AIN 2: track 111.6 -> 0.00 mm
- net A0: track 35.7 -> 146.9 mm
- net Net-(D1-K): track 75.4 -> 0.00 mm
- net AIN 1: track 85.5 -> 12.2 mm
- net D5(G): track 53.9 -> 5.11 mm
- net D6(B): track 53.7 -> 5.64 mm
- net D1: track 5.61 -> 48.2 mm
- net D2: track 7.85 -> 48.2 mm
- net Net-(Q1-B): track 5.61 -> 45.6 mm
- net A1: track 38.7 -> 0.00 mm
- net Net-(Q2-B): track 3.98 -> 38.8 mm
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Other:
- board text removed: "Katrin F. Cedric S. Linda S."
- board text removed: "Riesen SPS"

Commit message: dedee
Parts:
- moved D14 41.2 mm to (108.2, 117.6), turned to -90 degrees
- moved U1 6.38 mm to (138.2, 111.4)
- moved C2 4.35 mm to (138.2, 115.5)
- moved J1 3.25 mm to (182.9, 140.7)
- moved D11 3.18 mm to (142.5, 90.1)
- moved D15 3.18 mm to (142.5, 98.1)
- moved D9 3.18 mm to (142.5, 94.1)
- moved R19 3.18 mm to (128.6, 98.1)
- moved R14 3.18 mm to (128.5, 90.1)
- moved R16 3.18 mm to (128.5, 94.1)
Connections:
- A1 pad 20: A1 -> unconnected-(A1-A1-Pad20)
Routing:
- net +5V: track 314.6 -> 288.7 mm
- net Vin: track 41.4 -> 63.2 mm
- net GND: track 192.8 -> 208.9 mm
- net A0: track 146.9 -> 153.4 mm
- net Net-(D7-K): track 19.7 -> 23.2 mm
- net Net-(D13-K): track 11.3 -> 14.7 mm
- net GND1: track 118.1 -> 121.3 mm
- net NO 2: track 13.1 -> 16.4 mm
- net NC 2: track 11.7 -> 15.0 mm
- net NC 1: track 12.0 -> 15.3 mm
- net DI3: track 8.84 -> 12.1 mm
- net DI2: track 8.87 -> 12.1 mm
- net AIN 1: track 12.2 -> 15.4 mm
- net COM2: track 27.1 -> 30.4 mm
- net COM1: track 25.8 -> 29.1 mm
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